File: be2.kicad_pcb (KiCad board)
At the start: 2 copper layers, 50 x 30 mm, 32 parts, among them K1 CONN_01X03, K2 CONN_01X02, K3 CONN_01X01, U1 AD620A, U2 TL082, U3 TL082

Commit message: some changes, simu ...
Parts:
- removed G***: LOGO, logo:logo_phelma_32x21mm

Commit message: part2 + routing
Parts:
- added C11: 10n, Capacitors_SMD:C_1206, F.Cu at (137.9, 103.8)
- added C12: 10n, Capacitors_SMD:C_1206, F.Cu at (131.4, 109.2)
- added D100: LED, lib:KP-3216SRC-PRV, F.Cu at (164.0, 100.5)
- added D101: LED, lib:KP-3216SRC-PRV, F.Cu at (164.0, 107.5)
- added D102: LED, lib:KP-3216SRC-PRV, F.Cu at (164.0, 114.5)
- added D103: LED, lib:KP-3216SRC-PRV, F.Cu at (164.0, 121.5)
- added G***: LOGO, logo:logo_phelma_32x21mm, F.Cu at (137.0, 120.1)
- added K4: CONN_01X03, lib:Pin_Header_Straight_1x03_phelma, B.Cu at (121.5, 104.0)
- added K5: CONN_01X01, lib:Pin_Header_Straight_1x01_phelma, B.Cu at (121.5, 99.0)
- added R100: 1k, Resistors_SMD:R_1206, F.Cu at (161.7, 100.5)
- added R101: 1k, Resistors_SMD:R_1206, F.Cu at (161.7, 107.5)
- added R102: 1k, Resistors_SMD:R_1206, F.Cu at (161.7, 114.5)
- added R103: 1k, Resistors_SMD:R_1206, F.Cu at (161.7, 121.5)
- added R11: R_Small, Resistors_SMD:R_1206, F.Cu at (143.6, 113.2)
- added R12: R_Small, Resistors_SMD:R_1206, F.Cu at (143.6, 108.6)
- added R13: R_Small, Resistors_SMD:R_1206, F.Cu at (143.6, 104.0)
- added R6: 1K, Resistors_SMD:R_1206, F.Cu at (127.7, 105.9)
- added R7: 100K, Resistors_SMD:R_1206, F.Cu at (127.7, 101.3)
- added U100: LM311N, Housings_SOIC:SOIC-8_3.9x4.9mm_Pitch1.27mm, F.Cu at (156.7, 100.5)
- added U101: LM311N, Housings_SOIC:SOIC-8_3.9x4.9mm_Pitch1.27mm, F.Cu at (156.7, 107.5)
- added U102: LM311N, Housings_SOIC:SOIC-8_3.9x4.9mm_Pitch1.27mm, F.Cu at (156.7, 114.5)
- added U103: LM311N, Housings_SOIC:SOIC-8_3.9x4.9mm_Pitch1.27mm, F.Cu at (156.7, 121.5)
- added U4: TL082, Housings_SOIC:SOIC-8_3.9x4.9mm_Pitch1.27mm, F.Cu at (132.8, 104.2)
- added jp_close1: JP3, lib:JP_20mil, F.Cu at (147.3, 107.4)
- added jp_close2: JP3, lib:JP_20mil, F.Cu at (147.3, 111.3)
- moved C7 116.8 mm to (145.1, 90.3)
- moved R4 116.8 mm to (149.2, 70.2)
- moved R5 116.8 mm to (144.6, 70.2)
- moved U1 116.8 mm to (138.0, 82.5)
- moved C1 116.8 mm to (126.2, 75.0)
- moved C5 116.8 mm to (144.6, 67.8)
- moved D1 116.8 mm to (146.1, 79.4)
- moved D3 116.8 mm to (129.1, 87.9)
- moved D4 116.8 mm to (132.1, 84.3)
- moved D5 116.8 mm to (132.1, 81.2)
- moved D6 116.8 mm to (129.1, 77.2)
- moved JP2 116.8 mm to (153.9, 81.6)
- moved K1 116.8 mm to (121.5, 71.5)
- moved K2 116.8 mm to (121.5, 81.7)
- moved K3 116.8 mm to (121.5, 66.5)
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Connections:
- net /mean_out renamed /amp_in
Routing:
- net VCC: track 89.8 -> 281.3 mm, vias 0 -> 2
- net VSS: track 108.6 -> 229.8 mm, vias 0 -> 4
- net /amp_in: track 56.5 -> 101.5 mm, vias 0 -> 2
- net /amp_out: track 0.00 -> 39.3 mm, vias 0 -> 2
- net GND: track 122.4 -> 158.4 mm, vias 0 -> 1
- net /ref_1v_div_pi: track 0.00 -> 33.1 mm
- net /ref_10v_div_pi: track 0.00 -> 29.3 mm
- net /comp_in_x100: track 0.00 -> 25.6 mm
- net /comp_in_x1: track 0.00 -> 24.3 mm
- net Net-(D102-Pad1): track 0.00 -> 6.83 mm
- net Net-(D103-Pad1): track 0.00 -> 6.52 mm
- net Net-(D101-Pad1): track 0.00 -> 6.52 mm
- net Net-(D100-Pad1): track 0.00 -> 6.52 mm
- net Net-(R6-Pad1): track 0.00 -> 4.49 mm
- net Net-(D101-Pad2): track 0.00 -> 2.54 mm
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Other:
- board size 50 x 30 mm -> 50 x 62.5 mm
- net class Default: via_dia 0.6 -> 2; via_drill 0.4 -> 1
- net class power: via_dia 0.6 -> 2; via_drill 0.4 -> 1
- board text added: "F.Cu"
- board text added: "|i+|i-| |+|-|g|"

Commit message: mechanical drawing
Parts:
- moved C1 77.4 mm to (53.1, 49.5)
- moved C7 77.4 mm to (72.0, 64.8)
- moved JP2 77.4 mm to (80.8, 56.0)
- moved R4 77.4 mm to (76.1, 44.6)
- moved R5 77.4 mm to (71.5, 44.6)
- moved U1 77.4 mm to (64.9, 57.0)
- moved C10 77.4 mm to (66.8, 42.2)
- moved C2 77.4 mm to (51.8, 44.6)
- moved C3 77.4 mm to (66.4, 62.0)
- moved C4 77.4 mm to (63.4, 62.0)
- moved C5 77.4 mm to (71.5, 42.2)
- moved C6 77.4 mm to (80.7, 60.0)
- moved C8 77.4 mm to (61.0, 49.7)
- moved D1 77.4 mm to (73.0, 53.9)
- moved D2 77.4 mm to (80.1, 64.8)
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Other:
- board size 50 x 62.5 mm -> 130 x 30 mm
- board text added: "+15v [4]"
- board text added: "-15v [3]"
- board text added: "KA-001 module"
- board text added: "KA-002 module"
- board text added: "ground [2]"
- board text added: "in+ [5]"
- board text added: "in- [6]"
- board text added: "mean_in [1]"
- board text added: "mean_out [1]"
